File: PCB_Keyboard.kicad_pcb (KiCad board)
At the start: 2 copper layers, 0 parts

Commit message: roteamento
Parts:
- added C1: 1uF, Capacitor_SMD:C_0805_2012Metric, F.Cu at (68.2, 83.2)
- added C2: 0.1uF, Capacitor_SMD:C_0805_2012Metric, F.Cu at (73.8, 75.5)
- added C3: 0.1uF, Capacitor_SMD:C_0805_2012Metric, F.Cu at (85.7, 88.2)
- added C4: 0.1uF, Capacitor_SMD:C_0805_2012Metric, F.Cu at (81.7, 75.4)
- added C5: 0.1uF, Capacitor_SMD:C_0805_2012Metric, F.Cu at (72.3, 92.2)
- added C6: 22pF, Capacitor_SMD:C_0805_2012Metric, F.Cu at (82.5, 93.5)
- added C7: 22pF, Capacitor_SMD:C_0805_2012Metric, F.Cu at (75.7, 93.4)
- added D1: D_Small, Diode_SMD:D_SOD-123, F.Cu at (106.3, 72.9)
- added D2: D_Small, Diode_SMD:D_SOD-123, F.Cu at (126.0, 72.6)
- added D3: D_Small, Diode_SMD:D_SOD-123, F.Cu at (106.3, 93.0)
- added D4: D_Small, Diode_SMD:D_SOD-123, F.Cu at (126.0, 93.1)
- added F1: 500mA, Fuse:Fuse_1206_3216Metric, F.Cu at (80.3, 69.8)
- added MX1: MX-NoLED, MX_Alps_Hybrid:MX-Alps-Hybrid-1U, F.Cu at (98.2, 71.0)
- added MX2: MX-NoLED, MX_Alps_Hybrid:MX-Alps-Hybrid-1U, F.Cu at (117.8, 71.0)
- added MX3: MX-NoLED, MX_Alps_Hybrid:MX-Alps-Hybrid-1U, F.Cu at (98.2, 90.8)
- added MX4: MX-NoLED, MX_Alps_Hybrid:MX-Alps-Hybrid-1U, F.Cu at (117.9, 90.8)
- added R1: 10k, Resistor_SMD:R_0805_2012Metric, F.Cu at (85.6, 80.7)
- added R2: 22, Resistor_SMD:R_0805_2012Metric, F.Cu at (72.2, 70.5)
- added R3: 22, Resistor_SMD:R_0805_2012Metric, F.Cu at (69.3, 70.5)
- added R4: 10k, Resistor_SMD:R_0805_2012Metric, F.Cu at (68.7, 91.4)
- added SW1: SW_Push, random-keyboard-parts:SKQG-1155865, F.Cu at (69.0, 97.4)
- added U1: ATmega32U4-A, Package_QFP:TQFP-44_10x10mm_P0.8mm, F.Cu at (77.6, 83.4)
- added USB1: Molex-0548190589, random-keyboard-parts:Molex-0548190589, F.Cu at (70.3, 62.2)
- added Y1: 16MHz, Crystal:Crystal_SMD_3225-4Pin_3.2x2.5mm, F.Cu at (79.2, 93.5)
Routing:
- net GND: track 0.00 -> 99.6 mm, vias 0 -> 6
- net col1: track 0.00 -> 68.5 mm
- net row1: track 0.00 -> 48.9 mm
- net row0: track 0.00 -> 47.5 mm, vias 0 -> 2
- net col0: track 0.00 -> 44.8 mm, vias 0 -> 2
- net +5V: track 0.00 -> 28.3 mm
- net Net-(U1-D+): track 0.00 -> 13.2 mm
- net Net-(U1-~{RESET}): track 0.00 -> 12.9 mm
- net Net-(U1-D-): track 0.00 -> 11.9 mm
- net Net-(U1-XTAL2): track 0.00 -> 9.88 mm
- net Net-(D3-A): track 0.00 -> 9.49 mm
- net Net-(D4-A): track 0.00 -> 9.41 mm
- net Net-(D2-A): track 0.00 -> 9.15 mm
- net VCC: track 0.00 -> 9.12 mm
- net Net-(D1-A): track 0.00 -> 8.79 mm
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Other:
- board outline added: 65.9 x 41.3 mm

Commit message: fix de uma trilha que eu esqueci de colocar
Routing:
- net GND: track 99.6 -> 103.5 mm
Changed lines of the file:
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@@
+	)
+	(segment
+		(start 68.57425 82.6395)
+		(end 68.199 82.26425)
+		(width 0.2)
+		(layer "F.Cu")
+		(net 1)
 	)
 	(segment
@@
 		(width 0.2)
 		(layer "F.Cu")
+		(net 1)
+	)
+	(segment
+		(start 71.91375 82.6395)
+		(end 68.57425 82.6395)
+		(width 0.2)
+		(layer "F.Cu")

Commit message: GND Fill e Gerbers
Routing:
- added copper zone on F.Cu, net GND
Changed lines of the file:
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@@
 			(outputformat 1)
 			(mirror no)
-			(drillshape 1)
+			(drillshape 0)
 			(scaleselection 1)
-			(outputdirectory "")
+			(outputdirectory "Drill/")
 		)
 	)
@@
 		(net 20)
 	)
+	(zone
+		(net 1)
+		(net_name "GND")
+		(layer "F.Cu")
+		(hatch edge 0.5)
+		(connect_pads
+			(clearance 0.5)
+		)
+		(min_thickness 0.25)
+		(filled_areas_thickness no)
+		(fill yes
+			(thermal_gap 0.5)
+			(thermal_bridge_width 0.5)
+		)
+		(polygon
+			(pts
+				(xy 64.008 101.219) (xy 88.011 101.346) (xy 88.265 60.833) (xy 64.135 61.087)
+			)
+		)
+	)
 	(embedded_fonts no)
